File: HW/Main board/PullupCounter-MainBoard/PullupCounter-MainBoard.sch (KiCad schematic (older format))
At the start: 38 parts

Commit message: soon done
Parts:
- added C? (x3): 100n, symbol Device:C
- added C?: 100n, symbol Device:C_Small
- added R? (x3): 100K, symbol Device:R
- added R? (x3): 10K, symbol Device:R
- added ROT?: ROTARY-ENCODER-Ebay, symbol Peters:ROTARY-ENCODER-Ebay
- added U? (x4): 74HC14, symbol 74xx:74HC14
Connections:
- net labels added: encA, encB, encBTN
- wire segments 85 -> 110
Other:
- note added: "BTN needs to be double inverted"
- note added: "Rotary Encoder"

Commit message: Schematic and layout
Parts:
- added MH1, MH2, MH3, MH4: MountingHole, MountingHole:MountingHole_3.2mm_M3, symbol Mechanical:MountingHole
- BT1: renamed from BT?; footprint (none) -> Libs:Cheap_CR2032_holder
- C1, C10, C11, C12, C13, C14, C15, C16, C17, C18, C19, C2, C20, C21, C5, C6, C7, C8, C9: renamed from C?; footprint (none) -> Capacitor_SMD:C_0805_2012Metric_Pad1.15x1.40mm_HandSolder
- C22: renamed from C?; footprint (none) -> Capacitor_SMD:CP_Elec_10x10.5
- C3, C4: renamed from C?; footprint (none) -> Capacitor_Tantalum_SMD:CP_EIA-3528-12_Kemet-T_Pad1.50x2.35mm_HandSolder
- ISP1: renamed from ISP?; footprint Pin_Headers:Pin_Header_Straight_2x03_Pitch2.54mm -> Connector_PinSocket_2.54mm:PinSocket_2x03_P2.54mm_Vertical
- J1: renamed from J?; footprint (none) -> Connector_BarrelJack:BarrelJack_Horizontal
- J2: renamed from J?; footprint (none) -> Connector_PinHeader_2.54mm:PinHeader_1x06_P2.54mm_Vertical_SMD_Pin1Left
- J3: renamed from J?; footprint (none) -> Connector_RJ:RJ45_Amphenol_54602-x08_Horizontal
- R1, R10, R11, R2, R3, R4, R5, R6, R7, R8, R9: renamed from R?; footprint (none) -> Resistor_SMD:R_0805_2012Metric_Pad1.15x1.40mm_HandSolder
- ROT1: renamed from ROT?; footprint (none) -> Libs:ROTARY-ENCODER-Ebay
- SW1: renamed from SW?; footprint (none) -> Libs:PushBTN KSC241G
- U1: renamed from U?; footprint Housings_QFP:TQFP-32_7x7mm_Pitch0.8mm -> Package_QFP:TQFP-32_7x7mm_P0.8mm
- U3: renamed from U?; footprint TO_SOT_Packages_SMD:SOT-223 -> Package_TO_SOT_SMD:SOT-223
- U4: renamed from U?; footprint (none) -> Package_SO:SOIC-14_3.9x8.7mm_P1.27mm
- U5, U8: renamed from U?; footprint (none) -> Libs:8x8LEDArray
- U6, U7: renamed from U?; footprint Housings_SOIC:SOIC-8_3.9x4.9mm_Pitch1.27mm -> Package_SO:SOIC-8_3.9x4.9mm_P1.27mm
- Y1: renamed from Y?; footprint (none) -> Crystal:Crystal_SMD_HC49-SD_HandSoldering
- Y2: renamed from Y?; footprint (none) -> Crystal:Crystal_AT310_D3.0mm_L10.0mm_Horizontal
- gave numbers to parts that had none: 1

Commit message: Layout started
Need to committo a board size and hole pattern
Parts:
- removed ISP1: ISP-header, Connector_PinSocket_2.54mm:PinSocket_2x03_P2.54mm_Vertical, symbol pro-mini-rescue:ISP-header
- added J4: AVR-ISP-6, Connector_PinSocket_2.54mm:PinSocket_2x03_P2.54mm_Vertical, symbol Connector:AVR-ISP-6
- added MH5, MH6: StripsFäste, MountingHole:MountingHole_3.2mm_M3, symbol Mechanical:MountingHole
- added R12, R13: 4k7, Resistor_SMD:R_0805_2012Metric_Pad1.15x1.40mm_HandSolder, symbol Device:R
- added unit 7 of U4
- BT1: footprint Libs:Cheap_CR2032_holder -> Battery:BatteryHolder_MPD_BC2003_1x2032
- Y1: footprint Crystal:Crystal_SMD_HC49-SD_HandSoldering -> Crystal:Crystal_AT310_D3.0mm_L10.0mm_Horizontal
- Y2: footprint Crystal:Crystal_AT310_D3.0mm_L10.0mm_Horizontal -> Crystal:Crystal_SMD_HC49-SD_HandSoldering
Connections:
- wire segments 110 -> 126
- no-connect marks 7 -> 16
