File: HW/Sensor board/Sensor board/Sensor board.sch (KiCad schematic (older format))
At the start: 23 parts, among them J1 RJ45_Shielded, U1 Hc-SR04, U2 DS92LV010A, U3 DS92LV010A, U4 LM2937xMP

Commit message: fix
Parts:
- removed J1: RJ45_Shielded, Connector_RJ:RJ45_Amphenol_RJHSE5380, symbol Connector:RJ45_Shielded
- added J1: 8P8C, Connector_RJ:RJ45_Amphenol_54602-x08_Horizontal, symbol Connector:8P8C
- C8: footprint Capacitor_Tantalum_SMD:CP_EIA-3528-12_Kemet-T_Pad1.50x2.35mm_HandSolder -> Capacitor_Tantalum_SMD:CP_EIA-6032-20_AVX-F_Pad2.25x2.35mm_HandSolder
Connections:
- wire segments 31 -> 30
Changed lines of the file:
@@
 	1    0    0    -1
-$EndComp
-$Comp
-L Connector:RJ45_Shielded J1
-U 1 1 5B82F20B
-P 8150 3050
-F 0 "J1" H 7821 2998 50  0000 R CNN
-F 1 "RJ45_Shielded" H 7821 3089 50  0000 R CNN
-F 2 "Connector_RJ:RJ45_Amphenol_RJHSE5380" V 8150 3075 50  0001 C CNN
-F 3 "~" V 8150 3075 50  0001 C CNN
-	1    8150 3050
-	-1   0    0    1
-$EndComp
-$Comp
-L power:GND #PWR0113
-U 1 1 5B82F304
-P 8150 2450
-F 0 "#PWR0113" H 8150 2200 50  0001 C CNN
-F 1 "GND" H 8155 2277 50  0000 C CNN
-F 2 "" H 8150 2450 50  0001 C CNN
-F 3 "" H 8150 2450 50  0001 C CNN
-	1    8150 2450
-	1    0    0    1
 $EndComp
 Text GLabel 1750 3900 0    50   Input ~ 0
@@
 Text GLabel 1750 4000 0    50   Input ~ 0
 ECHO
-Wire Wire Line
-	8150 2450 8150 2550
 Text GLabel 7750 2750 0    50   Input ~ 0
 TRIG+
@@
 F 0 "C8" H 8918 2696 50  0000 L CNN
 F 1 "15u" H 8918 2605 50  0000 L CNN
-F 2 "Capacitor_Tantalum_SMD:CP_EIA-3528-12_Kemet-T_Pad1.50x2.35mm_HandSolder" H 8838 2500 50  0001 C CNN
+F 2 "Capacitor_Tantalum_SMD:CP_EIA-6032-20_AVX-F_Pad2.25x2.35mm_HandSolder" H 8838 2500 50  0001 C CNN
 F 3 "~" H 8800 2650 50  0001 C CNN
 	1    8800 2650
@@
 $EndComp
 $Comp
-L power:GND #PWR0132
-U 1 1 5B838FA3
+L power:VCC #PWR0132
+U 1 1 5B8392A5
 P 4500 1500
-F 0 "#PWR0132" H 4500 1250 50  0001 C CNN
-F 1 "GND" H 4505 1327 50  0000 C CNN
+F 0 "#PWR0132" H 4500 1350 50  0001 C CNN
+F 1 "VCC" H 4517 1673 50  0000 C CNN
 F 2 "" H 4500 1500 50  0001 C CNN
 F 3 "" H 4500 1500 50  0001 C CNN
@@
 $EndComp
 $Comp
-L power:GND #PWR0133
-U 1 1 5B838FDC
+L power:VCC #PWR0133
+U 1 1 5B8392DE
 P 5100 1500
-F 0 "#PWR0133" H 5100 1250 50  0001 C CNN
-F 1 "GND" H 5105 1327 50  0000 C CNN
+F 0 "#PWR0133" H 5100 1350 50  0001 C CNN
+F 1 "VCC" H 5117 1673 50  0000 C CNN
 F 2 "" H 5100 1500 50  0001 C CNN
 F 3 "" H 5100 1500 50  0001 C CNN
@@
 	1    0    0    -1
 $EndComp
+$Comp
+L Connector:8P8C J1
+U 1 1 5B839475
+P 8150 3050
+F 0 "J1" H 7820 3054 50  0000 R CNN
+F 1 "8P8C" H 7820 3145 50  0000 R CNN
+F 2 "Connector_RJ:RJ45_Amphenol_54602-x08_Horizontal" V 8150 3075 50  0001 C CNN
+F 3 "~" V 8150 3075 50  0001 C CNN
+	1    8150 3050
+	-1   0    0    1
+$EndComp
 $EndSCHEMATC
